File: Design/FLCU-Test-2/FLCU-Test-2.kicad_sch (KiCad schematic)
At the start: 57 parts, among them J1 ICSP, J2 UART, J3 0348260124, U1 ATmega328-AU, U2 ULN2003ADR, U3 MCP2515-xST, U4 TJR1443, U5 NCV4276B, Y1 CSTNE16M0V530000R0, Y2 8MHz

Commit message: Tentative Completion of Rev2 of FLCU / GEM  - Switch to TJR1443 CAN transceiver  - Smaller, more modern crystal for MCP2515  - Pulse-forming network to use sleep/wake functionality of TJR1443  - Switch from 12 to 16 pin connector to allow one additional analog input,    one digital pulse capture input, +5VOUT and signal ground  - Put CAN INT on an actual interrupt pin (lol)
This revision was done to correct some sleep/wake issues with Rev1, and to support it's use as a boost controller (with different FW)

 - Out - PWM Boost Control Solenoid
 - Out - PWM Electric Water Pump (Intercooler)
 - Out - Intercooler Fan Relay
 - DIn - Turbine speed
 - AIn - Manifold Pressure
 - AIn - Discharge Air Temperature
 - AIn - Intercooler Water Temperature
 - AIn - There was one more that I'm forgetting
Parts:
- removed D5, D6, D7, D8: 1N4148WS, Diode_SMD:D_SOD-323F, symbol Device:D
- added C17, C26: 100nF, Capacitor_SMD:C_0805_2012Metric_Pad1.18x1.45mm_HandSolder, symbol Device:C_Small
- added C21, C22, C23, C24: 100n, Capacitor_SMD:C_0805_2012Metric_Pad1.18x1.45mm_HandSolder, symbol Device:C_Small
- added D4, D5: MMBD4448HCQW, Package_TO_SOT_SMD:SOT-353_SC-70-5, symbol Diode:MMBD4448HCQW
- added R10, R11, R12, R13, R14, R15, R16, R9: 10k, Resistor_SMD:R_0805_2012Metric_Pad1.20x1.40mm_HandSolder, symbol Device:R_Small
- added R17: R, Resistor_SMD:R_0805_2012Metric, symbol Device:R
- added R18, R6, R7: 10k, Resistor_SMD:R_0805_2012Metric_Pad1.20x1.40mm_HandSolder, symbol Device:R
- added R25: 47k, Resistor_SMD:R_0805_2012Metric, symbol Device:R
- added R26: 10k, Resistor_SMD:R_0805_2012Metric, symbol Device:R
- C1: footprint Capacitor_SMD:C_0603_1608Metric -> Capacitor_SMD:C_0805_2012Metric_Pad1.18x1.45mm_HandSolder
- C13: renamed from C14; footprint Capacitor_SMD:C_0603_1608Metric -> Capacitor_SMD:C_0805_2012Metric_Pad1.18x1.45mm_HandSolder
- C14: renamed from C15; footprint Capacitor_SMD:C_0603_1608Metric -> Capacitor_SMD:C_0805_2012Metric_Pad1.18x1.45mm_HandSolder
- C2: renamed from C5; footprint Capacitor_SMD:C_0603_1608Metric -> Capacitor_SMD:C_0805_2012Metric_Pad1.18x1.45mm_HandSolder
- C20: renamed from C19; footprint Capacitor_SMD:C_0603_1608Metric -> Capacitor_SMD:C_0805_2012Metric_Pad1.18x1.45mm_HandSolder
- C3: renamed from C2; footprint Capacitor_SMD:C_0603_1608Metric -> Capacitor_SMD:C_0805_2012Metric_Pad1.18x1.45mm_HandSolder
- C4: renamed from C3; footprint Capacitor_SMD:C_0603_1608Metric -> Capacitor_SMD:C_0805_2012Metric_Pad1.18x1.45mm_HandSolder
- C5: renamed from C4; footprint Capacitor_SMD:C_0603_1608Metric -> Capacitor_SMD:C_0805_2012Metric_Pad1.18x1.45mm_HandSolder
- J3: value 0348260124 -> 0348260160; footprint Molex_34826:0348260120 -> Molex_34826:0348260160; symbol Connector_Generic:Conn_01x12 -> Connector_Generic:Conn_01x16
- R29: renamed from R14; footprint Resistor_SMD:R_0603_1608Metric -> Resistor_SMD:R_0805_2012Metric_Pad1.20x1.40mm_HandSolder
- R4: renamed from R?; footprint (none) -> Resistor_SMD:R_0805_2012Metric_Pad1.20x1.40mm_HandSolder
- R5: renamed from R15; footprint Resistor_SMD:R_0603_1608Metric -> Resistor_SMD:R_0805_2012Metric_Pad1.20x1.40mm_HandSolder
- Y1: value CSTNE16M0V530000R0 -> 16MHz; footprint Crystal:Resonator_SMD_muRata_CSTxExxV-3Pin_3.0x1.1mm -> Crystal:Resonator_SMD_Murata_CSTxExxV-3Pin_3.0x1.1mm_HandSoldering; Part (none) -> CSTNE16M0V530000R0
- Y2: footprint Crystal:Crystal_SMD_HC49-SD -> Crystal:Crystal_SMD_5032-4Pin_5.0x3.2mm; symbol Device:Crystal_Small -> Device:Crystal_GND24_Small
- renumbered C12 to C11, C16 to C12, C11 to C15, C13 to C16, C17 to C18, C18 to C19, C20 to C25, C21 to C27, D4 to D1, D1 to D2, D2 to D3, D3 to D6, R6 to R19, R7 to R20, R8 to R21, R9 to R22, R12 to R23, R13 to R24, R10 to R27, R11 to R28, R5 to R8
Connections:
- net Module-Voltage is gone; now on net Sub-Level: U1.25 (PC2)
- net +12V: now also U4.10 (Vbat); no longer U4.5 (Vio)
- net +12V_BATTERY: now also J3.7 (Pin_7); no longer J3.5 (Pin_5)
- net +12V_IGN: now also J3.8 (Pin_8), C24.1, D4.1 (A), R12.1; no longer J3.7 (Pin_7)
- net +5V: now also J3.15 (Pin_15), R19.1, R21.1, R27.1, U4.5 (Vio), R17.1, R26.1; no longer U4.10 (Vbat)
- net CAN_H: now also J3.3 (Pin_3); no longer J3.6 (Pin_6)
- net CAN_INT: now also U1.1 (PD3); no longer U1.11 (PD7)
- net Extra-Out: now also J3.9 (Pin_9); no longer J3.11 (Pin_11)
- net GND: now also J3.16 (Pin_16), Y2.2, Y2.4, C17.1, C26.1, R10.2, R11.2, R12.2, R13.2, R14.2, R15.2, R16.2, R18.2, R7.2, R9.2; no longer RN1.8 (R1.2)
- net Low-Level-Warning: now also C17.2; no longer C20.2
- net Low-Level-Warning-Out: now also J3.10 (Pin_10), C23.1, D4.5 (A), R11.1; no longer J3.8 (Pin_8)
- net Main-Level-Out: now also J3.11 (Pin_11), C22.1, D4.4 (A), R10.1; no longer J3.9 (Pin_9)
- net Main-Lvl: now also C13.2, U1.26 (PC3); no longer C14.2
- net SCK: no longer R5.1
- net Sub-Level: now also C14.2; no longer C13.2, U1.23 (PC0)
- net Sub-Level-Out: now also J3.12 (Pin_12), C21.1, D4.3 (A), R9.1; no longer J3.10 (Pin_10)
- net POSTFUSE: now reaches D2.2 (A2), D3.2 (A), F1.1
- net at C7.1, U3.9 (OSC1): now also Y2.3; no longer Y2.2
- net PWM3: now reaches U2.1 (I1), U2.2 (I2)
- net PWM3: now also U1.14 (PB2); no longer U1.10 (PD6)
- net PWM1: now reaches U2.3 (I3), U2.4 (I4)
- net PWM1: now also U1.13 (PB1); no longer U1.9 (PD5)
- net PWM2: now reaches U2.5 (I5), U2.6 (I6)
- net PWM2: now also U1.11 (PD7); no longer U1.1 (PD3)
- net D4: now reaches U2.7 (I7)
- net D4: now also U1.10 (PD6); no longer U1.32 (PD2)
- net at U1.2 (PD4): now also R5.1
- net Wake_Sense: now reaches U1.27 (PC4)
- net Wake_Sense: now also R6.2, R7.1
- net Low-Level-Warning-In renamed A3_In
- net A3_In: now also J3.14 (Pin_14); no longer J3.12 (Pin_12)
- net Main-Level-In renamed A1_In
- net A1_In: now also J3.6 (Pin_6); no longer J3.4 (Pin_4)
- net Sub-Level-In renamed A2_In
- net A2_In: now also J3.5 (Pin_5); no longer J3.3 (Pin_3)
- net VReg_EN renamed A4_In
- net A4_In: now also J3.4 (Pin_4), R17.2
- net WAKE renamed Wake_Pulse
- net Wake_Pulse: now also D5.2 (K), D5.2 (K), D5.2 (K), D5.2 (K), R18.1
- new net: C21.2, D5.3 (A), R13.1
- new net: C22.2, D5.4 (A), R14.1
- new net: C24.2, D5.1 (A), R16.1
- new net: C23.2, D5.5 (A), R15.1
- new net: D4.2 (K), D4.2 (K), D4.2 (K), D4.2 (K), R6.1
- new net D1_INT_In: J3.13 (Pin_13), R25.2, R26.2
- new net EXT_INT: C26.2, R25.1, U1.32 (PD2)
- new net Spare-Analog: C20.2, RN1.8 (R1.2), U1.23 (PC0)
- no-connect marks 10 -> 6
Other:
- moved on the sheet: C1, C10, C11, C12, C13, C14, C15, C16, C18, C19, C2, C20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
